Commit message: added cadrl_ros, working

File: src/onebot_description/urdf/onebot.urdf.xacro (robot description, xacro)
@@ -6,4 +6,5 @@
     <xacro:include filename="$(find onebot_description)/urdf/materials.urdf.xacro" />
     <xacro:include filename="$(find onebot_description)/urdf/onebot.urdf.gazebo" />
+    <!-- <xacro:include filename="$(find onebot_description)/urdf/macro.xacro" /> -->
     <xacro:arg name="mesh_enabled" default="false" />
     <xacro:arg name="robot_namespace" default="/"/>
@@ -50,4 +51,31 @@
     <child link="camera_left_link"/>
   </joint>
+  <link name="sensor_laser">
+    <inertial>
+        <origin xyz="0 0.6 0.2" rpy="0 0 0" />
+        <mass value="0.001" />
+        <inertia  ixx="${0.001*(3*0.04*0.04+0.1*0.1)/12}" ixy = "0" ixz = "0"
+            iyy="${0.001*(3*0.04*0.04+0.1*0.1)/12}" iyz = "0"
+            izz="${0.001*(0.04*0.04)/2}" />
+    </inertial>
+    <visual>
+        <origin xyz="0 0 0" rpy="0 0 0" />
+        <geometry>
+        <cylinder radius="0.05" length="0.1"/>
+        </geometry>
+        <material name="white" />
+    </visual>
+    <collision>
+        <origin xyz="0 0 0" rpy="0 0 0"/>
+        <geometry>
+        <cylinder radius="0.05" length="0.1"/>
+        </geometry>
+    </collision>
+    </link>
+    <joint name="joint_sensor_laser" type="fixed">
+    <origin xyz="-0.25 0 0.05" rpy="0 0 0"/>
+    <parent link="base_link"/>
+    <child link="sensor_laser"/>
+  </joint>
   <!-- Camera Left -->
   <link name="camera_left_link">

Commit message: ready for rehearsal

File: src/onebot_description/urdf/onebot.urdf.xacro (robot description, xacro)
@@ -53,5 +53,5 @@
   <link name="sensor_laser">
     <inertial>
-        <origin xyz="0 0.6 0.2" rpy="0 0 0" />
+        <origin xyz="0 0.6 1.2" rpy="0 0 0" />
         <mass value="0.001" />
         <inertia  ixx="${0.001*(3*0.04*0.04+0.1*0.1)/12}" ixy = "0" ixz = "0"
@@ -74,5 +74,5 @@
     </link>
     <joint name="joint_sensor_laser" type="fixed">
-    <origin xyz="-0.25 0 0.05" rpy="0 0 0"/>
+    <origin xyz="-0.25 0 0.151" rpy="0 0 0"/>
     <parent link="base_link"/>
     <child link="sensor_laser"/>

Commit message: ready for pre3

File: src/onebot_description/urdf/onebot.urdf.xacro (robot description, xacro)
@@ -47,5 +47,5 @@
   <joint name="camera_left_joint" type="fixed">
     <axis xyz="0 1 0" />
-    <origin xyz="${mono_cam_x_pos} -${mono_cam_y_pos} 0.035" rpy="0 0 -1.75"/>
+    <origin xyz="${mono_cam_x_pos} -${mono_cam_y_pos} 0.035" rpy="0 0 0"/>
     <parent link="base_link"/>
     <child link="camera_left_link"/>
